Commit message: working GUI, failed ROS2 config files

File: install/pegasus_arm_description/share/pegasus_arm_description/URDF/pegasus_arm.urdf.xacro (robot description, xacro)
@@ -10,4 +10,7 @@
       </geometry>
       <origin xyz="0 0 0.06" rpy="0 0 0"/>
+      <material name="blue">
+        <color rgba="0.0 0.0 1.0 1.0"/>
+      </material>
     </visual>
     <collision>
@@ -28,4 +31,7 @@
       <geometry><box size="0.12 0.12 0.08"/></geometry>
       <origin xyz="0 0 0.04" rpy="0 0 0"/>
+      <material name="red">
+        <color rgba="1.0 0.0 0.0 1.0"/>
+      </material>
     </visual>
     <collision>
@@ -44,4 +50,7 @@
       <geometry><box size="0.25 0.08 0.06"/></geometry>
       <origin xyz="0.125 0 0" rpy="0 0 0"/>
+      <material name="green">
+        <color rgba="0.0 1.0 0.0 1.0"/>
+      </material>
     </visual>
     <collision>
@@ -60,4 +69,7 @@
       <geometry><box size="0.22 0.06 0.05"/></geometry>
       <origin xyz="0.11 0 0" rpy="0 0 0"/>
+      <material name="yellow">
+        <color rgba="1.0 1.0 0.0 1.0"/>
+      </material>
     </visual>
     <collision>
@@ -76,4 +88,7 @@
       <geometry><box size="0.18 0.05 0.04"/></geometry>
       <origin xyz="0.09 0 0" rpy="0 0 0"/>
+      <material name="orange">
+        <color rgba="1.0 0.5 0.0 1.0"/>
+      </material>
     </visual>
     <collision>
@@ -92,4 +107,7 @@
       <geometry><cylinder radius="0.03" length="0.08"/></geometry>
       <origin xyz="0.04 0 0" rpy="0 1.5708 0"/>
+      <material name="purple">
+        <color rgba="0.5 0.0 1.0 1.0"/>
+      </material>
     </visual>
     <collision>
@@ -108,4 +126,7 @@
       <geometry><box size="0.06 0.08 0.02"/></geometry>
       <origin xyz="0.03 0 0" rpy="0 0 0"/>
+      <material name="gray">
+        <color rgba="0.5 0.5 0.5 1.0"/>
+      </material>
     </visual>
     <collision>
@@ -124,4 +145,7 @@
       <geometry><box size="0.04 0.06 0.08"/></geometry>
       <origin xyz="0.02 0 0.04" rpy="0 0 0"/>
+      <material name="black">
+        <color rgba="0.0 0.0 0.0 1.0"/>
+      </material>
     </visual>
     <collision>
@@ -141,5 +165,5 @@
     <origin xyz="0 0 0" rpy="0 0 0"/>
   </joint>
-  <!-- Joint 1 - Base rotation (360° rotation) -->
+  <!-- Joint 1 - Base rotation (360° rotation) - Start at 0 (no change) -->
   <joint name="joint1" type="revolute">
     <parent link="base_link"/>
@@ -150,56 +174,36 @@
     <safety_controller k_velocity="0.1" k_position="0.1"/>
     <dynamics damping="0.2" friction="0.3"/>
-    <hardware_interface>
-      <command_interface name="position"/>
-      <state_interface name="position"/>
-      <state_interface name="velocity"/>
-    </hardware_interface>
-  </joint>
-  <!-- Joint 2 - Shoulder joint (35° range) -->
+  </joint>
+  <!-- Joint 2 - Shoulder joint (35° range) - Start at -15° to lift arm up -->
   <joint name="joint2" type="revolute">
     <parent link="link1"/>
     <child link="link2"/>
-    <origin xyz="0 0 0.08" rpy="0 0 0"/>
+    <origin xyz="0 0 0.08" rpy="0 -0.26 0"/>  <!-- -15° initial position -->
     <axis xyz="0 1 0"/>
     <limit lower="-0.61" upper="0.61" velocity="1.0" effort="60.0"/>
     <safety_controller k_velocity="0.1" k_position="0.1"/>
     <dynamics damping="0.15" friction="0.2"/>
-    <hardware_interface>
-      <command_interface name="position"/>
-      <state_interface name="position"/>
-      <state_interface name="velocity"/>
-    </hardware_interface>
-  </joint>
-  <!-- Joint 3 - Elbow joint (100° range) -->
+  </joint>
+  <!-- Joint 3 - Elbow joint (100° range) - Start at -45° to bend elbow -->
   <joint name="joint3" type="revolute">
     <parent link="link2"/>
     <child link="link3"/>
-    <origin xyz="0.25 0 0" rpy="0 0 0"/>
+    <origin xyz="0.25 0 0" rpy="0 -0.785 0"/>  <!-- -45° initial position -->
     <axis xyz="0 1 0"/>
     <limit lower="-1.75" upper="1.75" velocity="1.0" effort="30.0"/>
     <safety_controller k_velocity="0.1" k_position="0.1"/>
     <dynamics damping="0.1" friction="0.15"/>
-    <hardware_interface>
-      <command_interface name="position"/>
-      <state_interface name="position"/>
-      <state_interface name="velocity"/>
-    </hardware_interface>
-  </joint>
-  <!-- Joint 4 - Forearm joint (75° range) -->
+  </joint>
+  <!-- Joint 4 - Forearm joint (75° range) - Start at -30° to continue bend -->
   <joint name="joint4" type="revolute">
     <parent link="link3"/>
     <child link="link4"/>
-    <origin xyz="0.22 0 0" rpy="0 0 0"/>
+    <origin xyz="0.22 0 0" rpy="0 -1.31 0"/><!-- -210° initial position -->
     <axis xyz="0 1 0"/>
     <limit lower="-1.31" upper="1.31" velocity="1.0" effort="30.0"/>
     <safety_controller k_velocity="0.1" k_position="0.1"/>
     <dynamics damping="0.1" friction="0.1"/>
-    <hardware_interface>
-      <command_interface name="position"/>
-      <state_interface name="position"/>
-      <state_interface name="velocity"/>
-    </hardware_interface>
-  </joint>
-  <!-- Joint 5 - Wrist rotation (360° rotation) -->
+  </joint>
+  <!-- Joint 5 - Wrist rotation (360° rotation) - Start at 0 (no change) -->
   <joint name="joint5" type="revolute">
     <parent link="link4"/>
@@ -210,9 +214,4 @@
     <safety_controller k_velocity="0.1" k_position="0.1"/>
     <dynamics damping="0.05" friction="0.05"/>
-    <hardware_interface>
-      <command_interface name="position"/>
-      <state_interface name="position"/>
-      <state_interface name="velocity"/>
-    </hardware_interface>
   </joint>
   <!-- Joint 6 - Gripper mounting (fixed) -->
@@ -232,10 +231,9 @@
     <hardware>
       <plugin>mock_components/GenericSystem</plugin>
-      <param name="example_param">example_value</param>
     </hardware>
     <joint name="joint1">
       <command_interface name="position">
         <param name="min">-6.28</param>
-        <param name="max"> 6.28</param>
+        <param name="max">6.28</param>
       </command_interface>
       <state_interface name="position"/>
@@ -245,5 +243,5 @@
       <command_interface name="position">
         <param name="min">-0.61</param>
-        <param name="max"> 0.61</param>
+        <param name="max">0.61</param>
       </command_interface>
       <state_interface name="position"/>
@@ -253,5 +251,5 @@
       <command_interface name="position">
         <param name="min">-1.75</param>
-        <param name="max"> 1.75</param>
+        <param name="max">1.75</param>
       </command_interface>
       <state_interface name="position"/>
@@ -261,5 +259,5 @@
       <command_interface name="position">
         <param name="min">-1.31</param>
-        <param name="max"> 1.31</param>
+        <param name="max">1.31</param>
       </command_interface>
       <state_interface name="position"/>
@@ -269,5 +267,5 @@
       <command_interface name="position">
         <param name="min">-6.28</param>
-        <param name="max"> 6.28</param>
+        <param name="max">6.28</param>
       </command_interface>
       <state_interface name="position"/>
@@ -281,49 +279,44 @@
     </plugin>
   </gazebo>
-  <!-- Transmissions for ros2_control -->
-  <transmission name="joint1_trans">
-    <type>transmission_interface/SimpleTransmission</type>
-    <joint name="joint1">
-      <hardwareInterface>hardware_interface/PositionJointInterface</hardwareInterface>
-    </joint>
-    <actuator name="joint1_motor">
-      <mechanicalReduction>3.7</mechanicalReduction>
-    </actuator>
-  </transmission>
-  <transmission name="joint2_trans">
-    <type>transmission_interface/SimpleTransmission</type>
-    <joint name="joint2">
-      <hardwareInterface>hardware_interface/PositionJointInterface</hardwareInterface>
-    </joint>
-    <actuator name="joint2_motor">
-      <mechanicalReduction>2.0</mechanicalReduction>
-    </actuator>
-  </transmission>
-  <transmission name="joint3_trans">
-    <type>transmission_interface/SimpleTransmission</type>
-    <joint name="joint3">
-      <hardwareInterface>hardware_interface/PositionJointInterface</hardwareInterface>
-    </joint>
-    <actuator name="joint3_motor">
-      <mechanicalReduction>1</mechanicalReduction>
-    </actuator>
-  </transmission>
-  <transmission name="joint4_trans">
-    <type>transmission_interface/SimpleTransmission</type>
-    <joint name="joint4">
-      <hardwareInterface>hardware_interface/PositionJointInterface</hardwareInterface>
-    </joint>
-    <actuator name="joint4_motor">
-      <mechanicalReduction>1</mechanicalReduction>
-    </actuator>
-  </transmission>
-  <transmission name="joint5_trans">
-    <type>transmission_interface/SimpleTransmission</type>
-    <joint name="joint5">
-      <hardwareInterface>hardware_interface/PositionJointInterface</hardwareInterface>
-    </joint>
-    <actuator name="joint5_motor">
-      <mechanicalReduction>1</mechanicalReduction>
-    </actuator>
-  </transmission>
+  <!-- Gazebo material properties for better visualization -->
+  <gazebo reference="base_link">
+    <material>Gazebo/Blue</material>
+    <mu1>0.2</mu1>
+    <mu2>0.2</mu2>
+  </gazebo>
+  <gazebo reference="link1">
+    <material>Gazebo/Red</material>
+    <mu1>0.2</mu1>
+    <mu2>0.2</mu2>
+  </gazebo>
+  <gazebo reference="link2">
+    <material>Gazebo/Green</material>
+    <mu1>0.2</mu1>
+    <mu2>0.2</mu2>
+  </gazebo>
+  <gazebo reference="link3">
+    <material>Gazebo/Yellow</material>
+    <mu1>0.2</mu1>
+    <mu2>0.2</mu2>
+  </gazebo>
+  <gazebo reference="link4">
+    <material>Gazebo/Orange</material>
+    <mu1>0.2</mu1>
+    <mu2>0.2</mu2>
+  </gazebo>
+  <gazebo reference="link5">
+    <material>Gazebo/Purple</material>
+    <mu1>0.2</mu1>
+    <mu2>0.2</mu2>
+  </gazebo>
+  <gazebo reference="link6">
+    <material>Gazebo/Grey</material>
+    <mu1>0.2</mu1>
+    <mu2>0.2</mu2>
+  </gazebo>
+  <gazebo reference="end_effector_link">
+    <material>Gazebo/Black</material>
+    <mu1>0.2</mu1>
+    <mu2>0.2</mu2>
+  </gazebo>
 </robot>
